File: Hardware/py32f002b/py32f002b.brd (EAGLE design)
At the start: 43.9 x 18.6 mm, 26 parts, among them IC1 PY32F002BF15P6TU, IC2 AP2114HA-3.3TRG1, J1 USB_MINI-B_SMT, Y1 DSC6083CI1A-350K000T

Commit message: Final Draft
Parts:
- moved R2 0.63 mm to (30.6, 14.1)
- moved C1 0.54 mm to (17.4, 4.32)
Routing:
- net +3V3: track 96.0 -> 95.3 mm
- net GND: vias 15 -> 16
