File: Hardware/py32f002bf15p6/KiCAD/py32f002bf15p6.kicad_pcb (KiCad board)
At the start: 2 copper layers, 45.7 x 22.9 mm, 28 parts, among them J5 Conn_01x04_Pin, J6 Conn_01x13_Pin, J7 Conn_01x13_Pin, J8 USB_B_Mini, SW0 SW_Push, U1 CH340K, U3 AP2114HA-3.3TRG1, U4 py32f002bf15p6, Y1 16Mhz Crystal

Commit message: Change silkscreen and update gerbers
Other:
- board text added: "JP2 - Connect SW0:B5"
- board text removed: "JP2 - Connect SW0:A6"
Changed lines of the file:
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@@
+		)
+	)
+	(gr_text "SW0"
+		(at 172.68 100.54 0)
+		(layer "F.SilkS")
+		(effects
+			(font
+				(size 0.7112 0.7112)
+				(thickness 0.1524)
+				(bold yes)
+			)
+			(justify bottom)
 		)
 	)
@@
 		)
 	)
-	(gr_text "JP2 - Connect SW0:A6"
+	(gr_text "JP2 - Connect SW0:B5"
 		(at 173.68 88.64 0)
 		(layer "B.SilkS")
